Commit message: updates

File: conveyor_description_pkg/urdf/conveyor.xacro (robot description, xacro)
@@ -80,5 +80,5 @@
             <origin xyz="${axisX * base_length/2}  ${axisY *base_length/2} 0" rpy="0 0 ${angle}" />
             <axis xyz="0 0 1" />
-            <limit effort="100" velocity="100" lower="${-M_PI/4}" upper="${M_PI/4}" />
+            <limit effort="100" velocity="100" lower="${-2*M_PI}" upper="${2*M_PI}" />
             <dynamics damping="0" friction="0" />
         </joint>
@@ -148,5 +148,5 @@
     </gazebo>
     <!-- Wheel 1 -->
-    <xacro:servo front="front" right="right" parent="base_link" axisX="1" axisY="1" angle="${-M_PI/4}"/>
+    <xacro:servo front="front" right="right" parent="base_link" axisX="1" axisY="1" angle="${-M_PI/4}"/> <!-- ${3*M_PI/4} -->
     <xacro:wheel fb="front" lr="right" parent="servo_front_right_link" translateX="0" translateY="0" translateZ="${-base_height-0.005}" flipY="1" flipX="0" />
     <!-- Wheel 2 -->

Commit message: update

File: conveyor_description_pkg/urdf/conveyor.xacro (robot description, xacro)
@@ -79,5 +79,5 @@
             <child link="servo_${front}_${right}_link" />
             <origin xyz="${axisX * base_length/2}  ${axisY *base_length/2} 0" rpy="0 0 ${angle}" />
-            <axis xyz="0 0 1" />
+            <axis xyz="0 0 1" rpy="0 0 0" />
             <limit effort="100" velocity="100" lower="${-2*M_PI}" upper="${2*M_PI}" />
             <dynamics damping="0" friction="0" />
@@ -149,15 +149,15 @@
     </gazebo>
     <!-- Wheel 1 -->
-    <xacro:servo front="front" right="right" parent="base_link" axisX="1" axisY="1" angle="${3*M_PI/4}"/> <!-- ${-M_PI/4} -->
-    <xacro:wheel fb="front" lr="right" parent="servo_front_right_link" translateX="0" translateY="0" translateZ="${-base_height-0.0075}" flipY="1" flipX="0" />
+    <xacro:servo front="front" right="left" parent="base_link" axisX="1" axisY="1" angle="${3*M_PI/4}"/> <!-- ${-M_PI/4} -->
+    <xacro:wheel fb="front" lr="left" parent="servo_front_left_link" translateX="0" translateY="0" translateZ="${-base_height-0.0075}" flipY="1" flipX="0" rot = "-1"/>
     <!-- Wheel 2 -->
-    <xacro:servo front="front" right="left" parent="base_link" axisX="1" axisY="-1" angle="${M_PI/4}" /> <!-- ${5*M_PI/4} -->
-    <xacro:wheel fb="front" lr="left" parent="servo_front_left_link" translateX="0" translateY="0" translateZ="${-base_height-0.0075}" flipY="1" flipX="1" />
+    <xacro:servo front="front" right="right" parent="base_link" axisX="1" axisY="-1" angle="${M_PI/4}" /> <!-- ${5*M_PI/4} -->
+    <xacro:wheel fb="front" lr="right" parent="servo_front_right_link" translateX="0" translateY="0" translateZ="${-base_height-0.0075}" flipY="1" flipX="1" rot = "1"/>
     <!-- Wheel 3 -->
-    <xacro:servo front="back" right="right" parent="base_link" axisX="-1" axisY="1" angle="${5*M_PI/4}" /> <!-- ${M_PI/4} -->
-    <xacro:wheel fb="back" lr="right" parent="servo_back_right_link" translateX="0" translateY="0" translateZ="${-base_height-0.0075}" flipY="1" flipX="0" />
+    <xacro:servo front="back" right="left" parent="base_link" axisX="-1" axisY="1" angle="${5*M_PI/4}" /> <!-- ${M_PI/4} -->
+    <xacro:wheel fb="back" lr="left" parent="servo_back_left_link" translateX="0" translateY="0" translateZ="${-base_height-0.0075}" flipY="1" flipX="0" rot = "-1"/>
     <!-- Wheel 4 -->
-    <xacro:servo front="back" right="left" parent="base_link" axisX="-1" axisY="-1" angle="${-M_PI/4}" /> <!-- ${3*M_PI/4} -->
-    <xacro:wheel fb="back" lr="left" parent="servo_back_left_link" translateX="0" translateY="0" translateZ="${-base_height-0.0075}" flipY="1" flipX="1" />
+    <xacro:servo front="back" right="right" parent="base_link" axisX="-1" axisY="-1" angle="${-M_PI/4}" /> <!-- ${3*M_PI/4} -->
+    <xacro:wheel fb="back" lr="right" parent="servo_back_right_link" translateX="0" translateY="0" translateZ="${-base_height-0.0075}" flipY="1" flipX="1" rot = "1"/>
     <!-- laser -->
     <link name="hokuyo_link">

File: conveyor_description_pkg/urdf/wheel.urdf.xacro (robot description, xacro)
@@ -14,5 +14,5 @@
       izz="${m*r*r/2}" />
   </xacro:macro>
-  <xacro:macro name="wheel" params="fb lr parent translateX translateY translateZ flipY flipX">
+  <xacro:macro name="wheel" params="fb lr parent translateX translateY translateZ flipY flipX rot">
     <!--fb : front, back ; lr: left, right -->
     <link name="${fb}_${lr}_wheel">
@@ -74,5 +74,5 @@
       <child link="${fb}_${lr}_wheel" />
       <origin xyz="${translateX} ${translateY} ${translateZ}" rpy="0 0 ${flipX*M_PI}" />
-      <axis xyz="0 1 0" rpy="0  0" />
+      <axis xyz="0 ${rot} 0" rpy="0  0" />
       <limit effort="100" velocity="100" />
       <joint_properties damping="0.0" friction="0.0" />

Commit message: refactor

File: conveyor_description_pkg/urdf/conveyor.xacro (robot description, xacro)
@@ -1,5 +1,5 @@
 <?xml version="1.0"?>
 <robot name="conveyor" xmlns:xacro="http://www.ros.org/wiki/xacro">
-    <xacro:include filename="$(find conveyor_description_pkg)/urdf/wheel.urdf.xacro" />
+    <xacro:include filename="$(find conveyor_description_pkg)/urdf/wheel_joints.urdf.xacro" />
     <!-- ros_control plugin -->
     <gazebo>
@@ -9,98 +9,7 @@
         </plugin>
     </gazebo>
-    <!-- Box Inertia -->
-    <xacro:macro name="box_inertia" params="m w h d">
-        <inertia ixx="${m / 12.0 * (d*d + h*h)}" ixy="0.0" ixz="0.0" iyy="${m / 12.0 * (w*w + h*h)}" iyz="0.0" izz="${m / 12.0 * (w*w + d*d)}" />
-    </xacro:macro>
-    <!-- Defining the colors used in this robot -->
-    <material name="Black">
-        <color rgba="0.0 0.0 0.0 1.0" />
-    </material>
-    <material name="Red">
-        <color rgba="0.8 0.0 0.0 1.0" />
-    </material>
-    <material name="White">
-        <color rgba="1.0 1.0 1.0 1.0" />
-    </material>
-    <material name="Blue">
-        <color rgba="0.0 0.0 0.8 1.0" />
-    </material>
-    <!-- PROPERTY LIST -->
-    <!--All units in m-kg-s-radians unit system -->
-    <xacro:property name="M_PI" value="3.1415926535897931" />
-    <xacro:property name="M_PI_2" value="1.570796327" />
-    <xacro:property name="DEG_TO_RAD" value="0.017453293" />
-    <!-- Main body radius and height -->
-    <!-- Main Body Cylinder base   -->
-    <xacro:property name="base_length" value="0.15" /> <!-- BOX -->
-    <xacro:property name="base_height" value="0.02" />
-    <xacro:property name="base_mass" value="10" /> <!-- in kg-->
-    <!-- caster wheel radius and height -->
-    <!-- caster wheel mass -->
-    <xacro:property name="servo_cube" value="0.015" />
-    <xacro:property name="servo_mass" value="2.5" /> <!-- in kg-->
-    <!-- Hokuyo Laser scanner -->
-    <xacro:property name="hokuyo_size" value="0.01 0.05 0.02" />
-    <xacro:macro name="servo" params="front right parent axisX axisY angle">
-        <!-- Servo link -->
-        <link name="servo_${front}_${right}_link">
-            <visual>
-                <origin xyz="0 0 0" rpy="${M_PI/2} 0 0" />
-                <geometry>
-                    <box size="${servo_cube} ${servo_cube} ${servo_cube}" />
-                </geometry>
-                <material name="Black" />
-            </visual>
-            <visual>
-                <origin xyz="0 ${servo_cube/2} ${-servo_cube}" rpy="${M_PI/2} 0 0" />
-                <geometry>
-                    <box size="${servo_cube} ${servo_cube*2} ${servo_cube/1.5}" />
-                </geometry>
-                <material name="Black" />
-            </visual>
-            <collision>
-                <origin xyz="0 ${servo_cube/2} ${-servo_cube}" rpy="${M_PI/2} 0 0" />
-                <geometry>
-                    <box size="${servo_cube} ${servo_cube*2} ${servo_cube/1.5}" />
-                </geometry>
-            </collision>
-            <inertial>
-                <mass value="${servo_mass}" />
-                <origin xyz="0 0 0" />
-                <xacro:box_inertia m="${servo_mass}" w="${servo_cube}" h="${servo_cube}" d="${servo_cube}" />
-                <!-- <inertia ixx="0.001" ixy="0.0" ixz="0.0"
-                    iyy="0.001" iyz="0.0"
-                    izz="0.001" /> -->
-            </inertial>
-        </link>
-        <!-- Servo joint -->
-        <joint name="servo_${front}_${right}_joint" type="revolute">
-            <parent link="${parent}" />
-            <child link="servo_${front}_${right}_link" />
-            <origin xyz="${axisX * base_length/2}  ${axisY *base_length/2} 0" rpy="0 0 ${angle}" />
-            <axis xyz="0 0 1" rpy="0 0 0" />
-            <limit effort="100" velocity="100" lower="${-2*M_PI}" upper="${2*M_PI}" />
-            <dynamics damping="0" friction="0" />
-        </joint>
-        <gazebo reference="servo_${front}_${right}_link">
-            <selfCollide>false</selfCollide>
-            <turnGravityOff>false</turnGravityOff>
-            <mu1>0.2</mu1>
-            <mu2>0.2</mu2>
-        </gazebo>
-        <!-- Servo transmission -->
-        <transmission name="tran_servo_${front}_${right}">
-            <type>transmission_interface/SimpleTransmission</type>
-            <joint name="servo_${front}_${right}_joint">
-                <hardwareInterface>hardware_interface/EffortJointInterface</hardwareInterface>
-            </joint>
-            <actuator name="servo_${front}_${right}_motor">
-                <hardwareInterface>hardware_interface/EffortJointInterface</hardwareInterface>
-                <mechanicalReduction>1</mechanicalReduction>
-            </actuator>
-        </transmission>
-    </xacro:macro>
     <!-- BASE-FOOTPRINT -->
-    <!-- base_footprint is a fictitious link(frame) that is on the ground right below base_link origin -->
+    <!-- base_footprint is a fictitious link(frame) that is on the ground right below base_link
+    origin -->
     <link name="base_footprint">
         <visual>
@@ -123,10 +32,12 @@
     </joint>
     <!-- BASE-LINK -->
-    <!--Actual body/chassis of the robot-->
+    <!--Actual
+    body/chassis of the robot-->
     <link name="base_link">
         <inertial>
             <mass value="${base_mass}" />
             <origin xyz="0 0 0" />
-            <xacro:box_inertia m="${base_mass}" w="${base_length}" h="${base_length}" d="${base_height}" />
+            <xacro:box_inertia m="${base_mass}" w="${base_length}" h="${base_length}"
+                d="${base_height}" />
         </inertial>
         <visual>
@@ -149,15 +60,23 @@
     </gazebo>
     <!-- Wheel 1 -->
-    <xacro:servo front="front" right="left" parent="base_link" axisX="1" axisY="1" angle="${3*M_PI/4}"/> <!-- ${-M_PI/4} -->
-    <xacro:wheel fb="front" lr="left" parent="servo_front_left_link" translateX="0" translateY="0" translateZ="${-base_height-0.0075}" flipY="1" flipX="0" rot = "-1"/>
+    <xacro:servo front="front" right="left" parent="base_link" axisX="1" axisY="1"
+        angle="${3*M_PI/4}" /> <!-- ${-M_PI/4} -->
+    <xacro:wheel fb="front" lr="left" parent="servo_front_left_link" translateX="0" translateY="0"
+        translateZ="${-base_height-0.0075}" flipY="1" flipX="0" rot="-1" />
     <!-- Wheel 2 -->
-    <xacro:servo front="front" right="right" parent="base_link" axisX="1" axisY="-1" angle="${M_PI/4}" /> <!-- ${5*M_PI/4} -->
-    <xacro:wheel fb="front" lr="right" parent="servo_front_right_link" translateX="0" translateY="0" translateZ="${-base_height-0.0075}" flipY="1" flipX="1" rot = "1"/>
+    <xacro:servo front="front" right="right" parent="base_link" axisX="1" axisY="-1"
+        angle="${M_PI/4}" /> <!-- ${5*M_PI/4} -->
+    <xacro:wheel fb="front" lr="right" parent="servo_front_right_link" translateX="0" translateY="0"
+        translateZ="${-base_height-0.0075}" flipY="1" flipX="1" rot="1" />
     <!-- Wheel 3 -->
-    <xacro:servo front="back" right="left" parent="base_link" axisX="-1" axisY="1" angle="${5*M_PI/4}" /> <!-- ${M_PI/4} -->
-    <xacro:wheel fb="back" lr="left" parent="servo_back_left_link" translateX="0" translateY="0" translateZ="${-base_height-0.0075}" flipY="1" flipX="0" rot = "-1"/>
+    <xacro:servo front="back" right="left" parent="base_link" axisX="-1" axisY="1"
+        angle="${5*M_PI/4}" /> <!-- ${M_PI/4} -->
+    <xacro:wheel fb="back" lr="left" parent="servo_back_left_link" translateX="0" translateY="0"
+        translateZ="${-base_height-0.0075}" flipY="1" flipX="0" rot="-1" />
     <!-- Wheel 4 -->
-    <xacro:servo front="back" right="right" parent="base_link" axisX="-1" axisY="-1" angle="${-M_PI/4}" /> <!-- ${3*M_PI/4} -->
-    <xacro:wheel fb="back" lr="right" parent="servo_back_right_link" translateX="0" translateY="0" translateZ="${-base_height-0.0075}" flipY="1" flipX="1" rot = "1"/>
+    <xacro:servo front="back" right="right" parent="base_link" axisX="-1" axisY="-1"
+        angle="${-M_PI/4}" /> <!-- ${3*M_PI/4} -->
+    <xacro:wheel fb="back" lr="right" parent="servo_back_right_link" translateX="0" translateY="0"
+        translateZ="${-base_height-0.0075}" flipY="1" flipX="1" rot="1" />
     <!-- laser -->
     <link name="hokuyo_link">
@@ -174,5 +93,5 @@
                 <box size="${hokuyo_size}" />
             </geometry>
-          </collision>
+        </collision>
     </link>
     <joint name="hokuyo_joint" type="fixed">

Commit message: update lidar

File: conveyor_description_pkg/urdf/conveyor.xacro (robot description, xacro)
@@ -84,5 +84,5 @@
             <origin xyz="0 0 0" rpy="0 0 0" />
             <geometry>
-                <box size="${hokuyo_size}" />
+                <cylinder radius = "${hokuyo_size}" length = "${hokuyo_size}"/>
             </geometry>
             <material name="Blue" />
@@ -91,10 +91,11 @@
             <origin xyz="0 0 0" rpy="0 0 0" />
             <geometry>
-                <box size="${hokuyo_size}" />
+                <cylinder radius = "${hokuyo_size}" length = "${hokuyo_size}"/>
             </geometry>
         </collision>
     </link>
     <joint name="hokuyo_joint" type="fixed">
-        <origin xyz="${base_length/2} 0 ${-base_height+0.005}" rpy="0 0 0" />
+        <!-- <origin xyz="${base_length/2} 0 ${-base_height+0.005}" rpy="0 0 0" /> -->
+        <origin xyz="0 0 ${base_height}" rpy="0 0 0" />
         <parent link="base_link" />
         <child link="hokuyo_link" />
@@ -106,5 +107,5 @@
             <origin xyz="${base_length/2} 0 ${-base_height+0.005}" rpy="0 0 " />
             <visualize>false</visualize>
-            <update_rate>40</update_rate>
+            <update_rate>10</update_rate>
             <ray>
                 <scan>
@@ -112,6 +113,6 @@
                         <samples>720</samples>
                         <resolution>1</resolution>
-                        <min_angle>-1.570796</min_angle>
-                        <max_angle>1.570796</max_angle>
+                        <min_angle>-3.141592</min_angle>
+                        <max_angle>3.141592</max_angle>
                     </horizontal>
                 </scan>

File: conveyor_description_pkg/urdf/wheel_joints.urdf.xacro (robot description, xacro)
@@ -129,5 +129,6 @@
   <xacro:property name="servo_mass" value="2.5" /> <!-- in kg-->
   <!-- Hokuyo Laser scanner -->
-  <xacro:property name="hokuyo_size" value="0.01 0.05 0.02" />
+  <!-- <xacro:property name="hokuyo_size" value="0.01 0.05 0.02" /> -->
+  <xacro:property name="hokuyo_size" value="0.02" />
   <xacro:macro name="servo" params="front right parent axisX axisY angle">
     <!-- Servo link -->

Commit message: update xacro

File: conveyor_description_pkg/urdf/conveyor.xacro (robot description, xacro)
@@ -1,4 +1,16 @@
 <?xml version="1.0"?>
 <robot name="conveyor" xmlns:xacro="http://www.ros.org/wiki/xacro">
+    <!-- PROPERTY LIST -->
+    <!-- Main Body Box -->
+    <xacro:property name="base_length" value="0.255" /> <!-- in m-->
+    <xacro:property name="base_height" value="0.04" /> <!-- in m-->
+    <xacro:property name="base_mass" value="10" /> <!-- in kg-->
+    <!-- caster wheel radius and height -->
+    <!-- caster wheel mass -->
+    <xacro:property name="servo_cube" value="0.03" /> <!-- in m-->
+    <xacro:property name="servo_mass" value="2.5" /> <!-- in kg-->
+    <!-- Hokuyo Laser scanner -->
+    <!-- <xacro:property name="hokuyo_size" value="0.01 0.05 0.02" /> -->
+    <xacro:property name="hokuyo_size" value="0.04" />
     <xacro:include filename="$(find conveyor_description_pkg)/urdf/wheel_joints.urdf.xacro" />
     <!-- ros_control plugin -->
@@ -62,21 +74,21 @@
     <xacro:servo front="front" right="left" parent="base_link" axisX="1" axisY="1"
         angle="${3*M_PI/4}" /> <!-- ${-M_PI/4} -->
-    <xacro:wheel fb="front" lr="left" parent="servo_front_left_link" translateX="0" translateY="0"
-        translateZ="${-base_height-0.0075}" flipY="1" flipX="0" rot="-1" />
+    <xacro:wheel fb="front" lr="left" parent="servo_front_left_link" translateX="0" translateY="-0.005"
+        translateZ="${-base_height-0.011}" flipY="1" flipX="0" rot="-1" />
     <!-- Wheel 2 -->
     <xacro:servo front="front" right="right" parent="base_link" axisX="1" axisY="-1"
         angle="${M_PI/4}" /> <!-- ${5*M_PI/4} -->
-    <xacro:wheel fb="front" lr="right" parent="servo_front_right_link" translateX="0" translateY="0"
-        translateZ="${-base_height-0.0075}" flipY="1" flipX="1" rot="1" />
+    <xacro:wheel fb="front" lr="right" parent="servo_front_right_link" translateX="0" translateY="-0.005"
+        translateZ="${-base_height-0.011}" flipY="1" flipX="1" rot="1" />
     <!-- Wheel 3 -->
     <xacro:servo front="back" right="left" parent="base_link" axisX="-1" axisY="1"
         angle="${5*M_PI/4}" /> <!-- ${M_PI/4} -->
-    <xacro:wheel fb="back" lr="left" parent="servo_back_left_link" translateX="0" translateY="0"
-        translateZ="${-base_height-0.0075}" flipY="1" flipX="0" rot="-1" />
+    <xacro:wheel fb="back" lr="left" parent="servo_back_left_link" translateX="0" translateY="-0.005"
+        translateZ="${-base_height-0.011}" flipY="1" flipX="0" rot="-1" />
     <!-- Wheel 4 -->
     <xacro:servo front="back" right="right" parent="base_link" axisX="-1" axisY="-1"
         angle="${-M_PI/4}" /> <!-- ${3*M_PI/4} -->
-    <xacro:wheel fb="back" lr="right" parent="servo_back_right_link" translateX="0" translateY="0"
-        translateZ="${-base_height-0.0075}" flipY="1" flipX="1" rot="1" />
+    <xacro:wheel fb="back" lr="right" parent="servo_back_right_link" translateX="0" translateY="-0.005"
+        translateZ="${-base_height-0.011}" flipY="1" flipX="1" rot="1" />
     <!-- laser -->
     <link name="hokuyo_link">
@@ -84,5 +96,5 @@
             <origin xyz="0 0 0" rpy="0 0 0" />
             <geometry>
-                <cylinder radius = "${hokuyo_size}" length = "${hokuyo_size}"/>
+                <cylinder radius="${hokuyo_size}" length="${hokuyo_size/2}" />
             </geometry>
             <material name="Blue" />
@@ -91,5 +103,5 @@
             <origin xyz="0 0 0" rpy="0 0 0" />
             <geometry>
-                <cylinder radius = "${hokuyo_size}" length = "${hokuyo_size}"/>
+                <cylinder radius="${hokuyo_size}" length="${hokuyo_size/2}" />
             </geometry>
         </collision>
@@ -97,5 +109,5 @@
     <joint name="hokuyo_joint" type="fixed">
         <!-- <origin xyz="${base_length/2} 0 ${-base_height+0.005}" rpy="0 0 0" /> -->
-        <origin xyz="0 0 ${base_height}" rpy="0 0 0" />
+        <origin xyz="0 0 ${base_height/2+hokuyo_size/4}" rpy="0 0 0" />
         <parent link="base_link" />
         <child link="hokuyo_link" />
@@ -105,5 +117,5 @@
         <turnGravityOff>false</turnGravityOff>
         <sensor type="ray" name="head_hokuyo_sensor">
-            <origin xyz="${base_length/2} 0 ${-base_height+0.005}" rpy="0 0 " />
+            <origin xyz="${base_length/2} 0 ${-base_height}" rpy="0 0 " />
             <visualize>false</visualize>
             <update_rate>10</update_rate>
@@ -118,5 +130,5 @@
                 </scan>
                 <range>
-                    <min>0.10</min>
+                    <min>0.1</min>
                     <max>20.0</max>
                     <resolution>0.001</resolution>

File: conveyor_description_pkg/urdf/wheel_joints.urdf.xacro (robot description, xacro)
@@ -1,5 +1,6 @@
 <?xml version="1.0"?>
 <robot name="wheel" xmlns:xacro="http://www.ros.org/wiki/xacro">
-  <!--All units in m-kg-s-radians unit system -->
+  <!--All
+  units in m-kg-s-radians unit system -->
   <xacro:property name="M_PI" value="3.1415926535897931" />
   <xacro:property name="M_PI_2" value="1.570796327" />
@@ -8,6 +9,6 @@
   <!-- ################ Wheels ####################################### -->
   <!-- ############################################################### -->
-  <xacro:property name="wheel_radius" value="0.015" />
-  <xacro:property name="wheel_height" value="0.0075" />
+  <xacro:property name="wheel_radius" value="0.03" /> <!-- in m-->
+  <xacro:property name="wheel_height" value="0.017" /> <!-- in m-->
   <xacro:property name="wheel_mass" value="5" /> <!-- in kg-->
   <xacro:property name="base_x_origin_to_wheel_origin" value="0" />
@@ -118,17 +119,4 @@
     <color rgba="0.0 0.0 0.8 1.0" />
   </material>
-  <!-- PROPERTY LIST -->
-  <!-- Main body radius and height -->
-  <!-- Main Body Cylinder base   -->
-  <xacro:property name="base_length" value="0.15" /> <!-- BOX -->
-  <xacro:property name="base_height" value="0.02" />
-  <xacro:property name="base_mass" value="10" /> <!-- in kg-->
-  <!-- caster wheel radius and height -->
-  <!-- caster wheel mass -->
-  <xacro:property name="servo_cube" value="0.015" />
-  <xacro:property name="servo_mass" value="2.5" /> <!-- in kg-->
-  <!-- Hokuyo Laser scanner -->
-  <!-- <xacro:property name="hokuyo_size" value="0.01 0.05 0.02" /> -->
-  <xacro:property name="hokuyo_size" value="0.02" />
   <xacro:macro name="servo" params="front right parent axisX axisY angle">
     <!-- Servo link -->
