Commit message: camera rotation

File: conveyor_description_pkg/urdf/camera.xacro (robot description, xacro)
@@ -1,45 +1,70 @@
 <?xml version="1.0"?>
-<robot xmlns:xacro="http://www.ros.org/wiki/xacro" >
-    <joint name="camera_joint" type="fixed">
-        <parent link="base_link"/>
-        <child link="camera_link"/>
-        <origin xyz="0 0 0.1" rpy="0 0 0"/>
-    </joint>
-    <link name="camera_link">
-        <visual>
-            <geometry>
-                <box size="0.010 0.03 0.03"/>
-            </geometry>
-            <material name="red"/>
-        </visual>
-    </link>
-    <joint name="camera_optical_joint" type="fixed">
-        <parent link="camera_link"/>
-        <child link="camera_link_optical"/>
-        <origin xyz="0 0 0" rpy="${-pi/2} 0 ${-pi/2}"/>
-    </joint>
-    <link name="camera_link_optical"></link>
-    <gazebo reference="camera_link">
-        <material>Gazebo/Red</material>
-        <sensor name="camera" type="camera">
-            <pose> 0 0 0 0 0 0 </pose>
-            <visualize>true</visualize>
-            <update_rate>10</update_rate>
-            <camera>
-                <horizontal_fov>1.089</horizontal_fov>
-                <image>
-                    <format>R8G8B8</format>
-                    <width>640</width>
-                    <height>480</height>
-                </image>
-                <clip>
-                    <near>0.05</near>
-                    <far>8.0</far>
-                </clip>
-            </camera>
-            <plugin name="camera_controller" filename="libgazebo_ros_camera.so">
-                <frame_name>camera_link_optical</frame_name>
-            </plugin>
-        </sensor>
-    </gazebo>
+<robot xmlns:xacro="http://www.ros.org/wiki/xacro">
+    <xacro:macro name="camera" params="base_link">
+        <joint name="camera_joint" type="revolute">
+            <parent link="${base_link}" />
+            <child link="camera_link" />
+            <origin xyz="0 0 0.1" rpy="0 0 0" />
+            <axis xyz="0 0 1" />
+            <limit lower="-3.14" upper="3.14" effort="50" velocity="10" />
+        </joint>
+        <link name="camera_link">
+            <visual>
+                <geometry>
+                    <box size="0.010 0.03 0.03" />
+                </geometry>
+                <material name="red" />
+            </visual>
+            <inertial>
+                <origin xyz="0 0 0" rpy="0 0 0"/>
+                <mass value="0.5"/>
+                <inertia
+                  ixx="1.05"  ixy="0.00"  ixz="0.00"
+                  iyx="0.00"  iyy="1.05"  iyz="0.00"
+                  izx="0.00"  izy="0.00"  izz="1.05"
+                />
+              </inertial>
+        </link>
+        <joint name="camera_optical_joint" type="fixed">
+            <parent link="camera_link" />
+            <child link="camera_link_optical" />
+            <origin xyz="0 0 0" rpy="${-pi/2} 0 ${-pi/2}" />
+        </joint>
+        <link name="camera_link_optical">
+        </link>
+        <gazebo reference="camera_link">
+            <material>Gazebo/Red</material>
+            <sensor name="camera" type="camera">
+                <pose> 0 0 0 0 0 0 </pose>
+                <visualize>true</visualize>
+                <update_rate>10</update_rate>
+                <camera>
+                    <horizontal_fov>1.089</horizontal_fov>
+                    <image>
+                        <format>R8G8B8</format>
+                        <width>640</width>
+                        <height>480</height>
+                    </image>
+                    <clip>
+                        <near>0.05</near>
+                        <far>8.0</far>
+                    </clip>
+                </camera>
+                <plugin name="camera_controller" filename="libgazebo_ros_camera.so">
+                    <frame_name>camera_link_optical</frame_name>
+                </plugin>
+            </sensor>
+        </gazebo>
+        <!-- Transmission -->
+        <transmission name="camera_tran">
+            <type>transmission_interface/SimpleTransmission</type>
+            <joint name="camera_joint">
+              <hardwareInterface>hardware_interface/EffortJointInterface</hardwareInterface>
+            </joint>
+            <actuator name="camera_joint_motor">
+              <hardwareInterface>hardware_interface/EffortJointInterface</hardwareInterface>
+              <mechanicalReduction>1</mechanicalReduction>
+            </actuator>
+          </transmission>
+    </xacro:macro>
 </robot>

File: conveyor_description_pkg/urdf/conveyor_camera.xacro (robot description, xacro)
@@ -97,4 +97,5 @@
         translateZ="${-base_height-0.011}" flipY="1" flipX="1" rot="1" />
     <!-- Camera -->
+    <xacro:camera base_link="base_link"/>
     <gazebo>
         <plugin name="p3d_base_controller" filename="libgazebo_ros_p3d.so">

Commit message: d435i revolute link

File: conveyor_description_pkg/urdf/camera.xacro (robot description, xacro)
@@ -17,12 +17,12 @@
             </visual>
             <inertial>
-                <origin xyz="0 0 0" rpy="0 0 0"/>
-                <mass value="0.5"/>
+                <origin xyz="0 0 0" rpy="0 0 0" />
+                <mass value="0.5" />
                 <inertia
-                  ixx="1.05"  ixy="0.00"  ixz="0.00"
-                  iyx="0.00"  iyy="1.05"  iyz="0.00"
-                  izx="0.00"  izy="0.00"  izz="1.05"
+                    ixx="1.05" ixy="0.00" ixz="0.00"
+                    iyx="0.00" iyy="1.05" iyz="0.00"
+                    izx="0.00" izy="0.00" izz="1.05"
                 />
-              </inertial>
+            </inertial>
         </link>
         <joint name="camera_optical_joint" type="fixed">
@@ -60,11 +60,11 @@
             <type>transmission_interface/SimpleTransmission</type>
             <joint name="camera_joint">
-              <hardwareInterface>hardware_interface/EffortJointInterface</hardwareInterface>
+                <hardwareInterface>hardware_interface/EffortJointInterface</hardwareInterface>
             </joint>
             <actuator name="camera_joint_motor">
-              <hardwareInterface>hardware_interface/EffortJointInterface</hardwareInterface>
-              <mechanicalReduction>1</mechanicalReduction>
+                <hardwareInterface>hardware_interface/EffortJointInterface</hardwareInterface>
+                <mechanicalReduction>1</mechanicalReduction>
             </actuator>
-          </transmission>
+        </transmission>
     </xacro:macro>
 </robot>

File: conveyor_description_pkg/urdf/conveyor_multi_camera.xacro (robot description, xacro)
@@ -14,9 +14,7 @@
     <xacro:property name="hokuyo_size" value="0.04" />
     <xacro:include filename="$(find conveyor_description_pkg)/urdf/wheel_joints.urdf.xacro" />
-    <xacro:include filename="$(find conveyor_description_pkg)/urdf/camera.xacro" />
     <!-- ros_control plugin -->
     <gazebo>
         <plugin name="gazebo_ros_control" filename="libgazebo_ros_control.so">
-            <robotNamespace>/conveyor</robotNamespace>
             <robotSimType>gazebo_ros_control/DefaultRobotHWSim</robotSimType>
         </plugin>
@@ -96,31 +94,59 @@
         translateY="-0.005"
         translateZ="${-base_height-0.011}" flipY="1" flipX="1" rot="1" />
-    <!-- Camera RGB -->
-    <!-- <xacro:camera base_link="base_link"/> -->
-    <!-- Revolute joint -->
-    <link name="camera_revolute_link"></link>
-    <joint name="camera_joint" type="revolute">
+    <!-- laser -->
+    <!-- <link name="hokuyo_link">
+        <visual>
+            <origin xyz="0 0 0" rpy="0 0 0" />
+            <geometry>
+                <cylinder radius="${hokuyo_size}" length="${hokuyo_size/2}" />
+            </geometry>
+            <material name="Blue" />
+        </visual>
+        <collision>
+            <origin xyz="0 0 0" rpy="0 0 0" />
+            <geometry>
+                <cylinder radius="${hokuyo_size}" length="${hokuyo_size/2}" />
+            </geometry>
+        </collision>
+    </link>
+    <joint name="hokuyo_joint" type="fixed">
+        <origin xyz="0 0 ${base_height/2+hokuyo_size/4}" rpy="0 0 0" />
         <parent link="base_link" />
-        <child link="camera_revolute_link" />
-        <origin xyz="0 0 0" rpy="0 0 0" />
-        <axis xyz="0 0 1" />
-        <limit lower="-3.14" upper="3.14" effort="50" velocity="10" />
+        <child link="hokuyo_link" />
     </joint>
-    <!-- Transmission joint camera -->
-    <transmission name="camera_tran">
-        <type>transmission_interface/SimpleTransmission</type>
-        <joint name="camera_joint">
-            <hardwareInterface>hardware_interface/EffortJointInterface</hardwareInterface>
-        </joint>
-        <actuator name="camera_joint_motor">
-            <hardwareInterface>hardware_interface/EffortJointInterface</hardwareInterface>
-            <mechanicalReduction>1</mechanicalReduction>
-        </actuator>
-    </transmission>
+    <gazebo reference="hokuyo_link">
+        <material>Gazebo/Blue</material>
+        <turnGravityOff>false</turnGravityOff>
+        <sensor type="ray" name="head_hokuyo_sensor">
+            <origin xyz="${base_length/2} 0 ${-base_height}" rpy="0 0 " />
+            <visualize>false</visualize>
+            <update_rate>10</update_rate>
+            <ray>
+                <scan>
+                    <horizontal>
+                        <samples>360</samples>
+                        <resolution>1</resolution>
+                        <min_angle>-3.141592</min_angle>
+                        <max_angle>3.141592</max_angle>
+                    </horizontal>
+                </scan>
+                <range>
+                    <min>0.1</min>
+                    <max>20.0</max>
+                    <resolution>0.001</resolution>
+                </range>
+            </ray>
+            <plugin name="gazebo_ros_head_hokuyo_controller" filename="libgazebo_ros_laser.so">
+                <topicName>/scan</topicName>
+                <frameName>hokuyo_link</frameName>
+            </plugin>
+        </sensor>
+    </gazebo> -->
     <!-- Camera RGBD realsense d435i -->
     <!-- github: https://github.com/m-tartari/realsense_gazebo_description?tab=readme-ov-file -->
-    <xacro:include filename="$(find realsense_gazebo_description)/urdf/_d435i.urdf.xacro" />
-    <xacro:sensor_d435i parent="camera_revolute_link" name="D435i_camera" topics_ns="D435i_camera">
-        <origin xyz="0.0 0.0 0.1" rpy="0.0 0.0 0.0" />
+    <xacro:arg name="robotns" default="conveyor" />
+    <xacro:include filename="$(find realsense_gazebo_description)/urdf/_d435i.urdf.xacro"/>
+    <xacro:sensor_d435i parent="base_link" name="/$(arg robotns)/D435i_camera" topics_ns="$(arg robotns)/D435i_camera">
+      <origin xyz="0.0 0.0 0.1" rpy="0.0 0.0 0.0"/>
     </xacro:sensor_d435i>
     <gazebo>
