Commit message: multi camera fix

File: conveyor_description_pkg/urdf/conveyor_multi_camera.xacro (robot description, xacro)
@@ -143,9 +143,29 @@
         </sensor>
     </gazebo> -->
+    <!-- Revolute joint -->
+    <link name="camera_revolute_link"></link>
+    <joint name="camera_joint" type="revolute">
+        <parent link="base_link" />
+        <child link="camera_revolute_link" />
+        <origin xyz="0 0 0" rpy="0 0 0" />
+        <axis xyz="0 0 1" />
+        <limit lower="-3.14" upper="3.14" effort="50" velocity="10" />
+    </joint>
+    <!-- Transmission joint camera -->
+    <transmission name="camera_tran">
+        <type>transmission_interface/SimpleTransmission</type>
+        <joint name="camera_joint">
+            <hardwareInterface>hardware_interface/EffortJointInterface</hardwareInterface>
+        </joint>
+        <actuator name="camera_joint_motor">
+            <hardwareInterface>hardware_interface/EffortJointInterface</hardwareInterface>
+            <mechanicalReduction>1</mechanicalReduction>
+        </actuator>
+    </transmission>
     <!-- Camera RGBD realsense d435i -->
     <!-- github: https://github.com/m-tartari/realsense_gazebo_description?tab=readme-ov-file -->
     <xacro:arg name="robotns" default="conveyor" />
     <xacro:include filename="$(find realsense_gazebo_description)/urdf/_d435i.urdf.xacro"/>
-    <xacro:sensor_d435i parent="base_link" name="/$(arg robotns)/D435i_camera" topics_ns="$(arg robotns)/D435i_camera">
+    <xacro:sensor_d435i parent="camera_revolute_link" name="/$(arg robotns)/D435i_camera" topics_ns="$(arg robotns)/D435i_camera">
       <origin xyz="0.0 0.0 0.1" rpy="0.0 0.0 0.0"/>
     </xacro:sensor_d435i>

Commit message: Update conveyor_multi_camera.xacro

File: conveyor_description_pkg/urdf/conveyor_multi_camera.xacro (robot description, xacro)
@@ -70,4 +70,35 @@
         <turnGravityOff>false</turnGravityOff>
     </gazebo>
+    <!-- palla -->
+    <link name="ball_link">
+        <inertial>
+            <mass value="0.0000000001" />
+            <origin xyz="0 0 0" />
+            <xacro:box_inertia m="0.0000000001" w="0.0000000001" h="0.0000000001"
+                d="0.0000000001" />
+        </inertial>
+        <visual>
+            <origin xyz="0 0 0" rpy="0 0 0" />
+            <geometry>
+                <sphere radius="0.1"/>
+            </geometry>
+            <material name="White" />
+        </visual>
+        <collision>
+            <origin xyz="0 0 0" rpy="0 0 0 " />
+            <geometry>
+                <sphere radius="0.0000000001"/>
+            </geometry>
+        </collision>
+    </link>
+    <gazebo reference="ball_link">
+        <material>Gazebo/Red</material>
+        <turnGravityOff>false</turnGravityOff>
+    </gazebo>
+    <joint name="ball_link" type="fixed">
+        <origin xyz="-0.2 0  0" rpy="0 0 0" />
+        <parent link="base_link" />
+        <child link="ball_link" />
+    </joint>
     <!-- Wheel 1 -->
     <xacro:servo front="front" right="left" parent="base_link" axisX="1" axisY="1"
